Commit message: Fix openarm_v10_right_arm_proper.xml duplicate keyframes
Removed duplicate pose1 and extended keyframe definitions that were
causing MuJoCo XML parsing to fail (ros2_control_node exit -6)

File: mujoco_models/openarm_v10.urdf (robot description, URDF)
Before this commit: robot openarm, 8 links, 7 joints
Joints:
- joint openarm_joint1: limit lower=-1.396263 upper=3.490659 effort=40 velocity=16.754666 -> lower=-1.396263 upper=3.490659 effort=200 velocity=16.754666
- joint openarm_joint2: limit lower=-1.745329 upper=1.745329 effort=40 velocity=16.754666 -> lower=-1.745329 upper=1.745329 effort=200 velocity=16.754666
- joint openarm_joint3: limit lower=-1.570796 upper=1.570796 effort=27 velocity=5.445426 -> lower=-1.570796 upper=1.570796 effort=150 velocity=5.445426
- joint openarm_joint4: limit lower=0.0 upper=2.443461 effort=27 velocity=5.445426 -> lower=0.0 upper=2.443461 effort=150 velocity=5.445426
- joint openarm_joint5: limit lower=-1.570796 upper=1.570796 effort=7 velocity=20.943946 -> lower=-1.570796 upper=1.570796 effort=50 velocity=20.943946
- joint openarm_joint6: limit lower=-0.785398 upper=0.785398 effort=7 velocity=20.943946 -> lower=-0.785398 upper=0.785398 effort=50 velocity=20.943946
- joint openarm_joint7: limit lower=-1.570796 upper=1.570796 effort=7 velocity=20.943946 -> lower=-1.570796 upper=1.570796 effort=50 velocity=20.943946
